File: hardware/cell-simulator.kicad_pcb (KiCad board)
At the start: 4 copper layers, 210 x 130 mm, 210 parts, among them CN1 IDC-SMD_16P-P2.54_Z-S23032101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, CN2 39-28-8020, P1 CONN-SMD_20P-P2.54_B-3000N20P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, Q1 TO255P460X1020X2008-3P, Q2 TO255P460X1020X2008-3P, Q3 TO255P460X1020X2008-3P, Q4 TO255P460X1020X2008-3P, U1 SOIC127P600X175-8N, U10 LM2904BQDRQ1, U11 LM2904BQDRQ1, U12 QFP50P1600X1600X160-100N, U13 KTW7, U14 KTW7, U15 KTW7, U16 KTW7, U17 SOT95P280X145-5N, U18 SOT-223_L6.5-W3.5-P2.30-LS7.0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, U19 URAXXXXYMD-10WR3, U2 QFP50P1200X1200X160-64N, U20 HEATSINK-TH_L23.5-W16.0-P18.0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, U21 HEATSINK-TH_L23.5-W16.0-P18.0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, U22 HEATSINK-TH_L23.5-W16.0-P18.0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, U23 HEATSINK-TH_L23.5-W16.0-P18.0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, U3 LM2904BQDRQ1, U4 LM2904BQDRQ1, U5 URBXXXXYMD-10WR3, U6 URBXXXXYMD-10WR3, U7 URBXXXXYMD-10WR3, U8 URBXXXXYMD-10WR3, U9 URAXXXXYMD-10WR3, X1 DSUB-TH_DMR-9S, Y1 ABLS-12.000MHZ-B2

Commit message: update OP amp circuit, update PCB.
Parts:
- removed R1, R26, R38, R54, R7: LC-0603_R, LC-0603_R
- removed R15, R28, R40, R9: R1210, R1210
Connections:
- R2 pad 1: GND1 -> C1I
- R27 pad 1: GND4 -> C4I
- R29 pad 2: $$$1477 -> C4
- R39 pad 1: GND3 -> C3I
- R41 pad 2: $$$1485 -> C3
- R6 pad 2: $$$10062 -> C1
- R8 pad 1: GND2 -> C2I
- RN4 pad 5: BUSY -> CAN1_TX
- RN4 pad 6: CHIPSELECT# -> CAN1_RX
- U1 pad 1: CAN1_RX -> CAN1_TX
- U1 pad 4: CAN1_TX -> CAN1_RX
- U12 pad 70: CAN1_RX -> CHIPSELECT#
- U12 pad 71: CAN1_TX -> BUSY
Routing:
- net CHIPSELECT#: track 23.7 -> 41.7 mm, vias 2 -> 3
- net BUSY: track 22.6 -> 40.6 mm, vias 2 -> 3
- net CAN1_RX: track 19.1 -> 37.1 mm
- net CAN1_TX: track 23.6 -> 39.3 mm
- net C1I: track 127.9 -> 138.6 mm
- net C4: track 250.2 -> 260.8 mm, vias 3 -> 5
- net C3I: track 71.9 -> 82.3 mm
- net C2: track 179.6 -> 190.0 mm, vias 3 -> 5
- net C4I: track 64.1 -> 74.4 mm
- net C2I: track 60.6 -> 70.7 mm
- net C3: track 213.4 -> 223.3 mm, vias 3 -> 5
- net C1: track 153.3 -> 162.3 mm, vias 3 -> 5
- net GND4: track 240.1 -> 237.0 mm, vias 63 -> 60
- net GND1: track 170.1 -> 167.0 mm
- net GND3: track 199.8 -> 196.7 mm, vias 64 -> 61
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