File: hardware/cell-simulator.kicad_sch (KiCad schematic)
At the start: 198 parts

Commit message: refactoring.
Parts:
- removed BEAD1: (no value), symbol Analog Processing-altium-import:0_0
- removed C1, C11, C12, C2, C5, C6, C8, C9: (no value), symbol Analog Processing-altium-import:1_220u
- removed C10, C3, C4, C7: (no value), symbol Analog Processing-altium-import:1_22u
- removed C13, C15, C17, C19, C21, C22, C23, C24: (no value), symbol Analog Processing-altium-import:1_100n
- removed C14, C16, C18, C20: (no value), symbol Analog Processing-altium-import:2_100n
- removed C26, C53, C75, C76: (no value), symbol Analog Processing-altium-import:0_10u
- removed C27: (no value), symbol Analog Processing-altium-import:1_10nF
- removed C28: (no value), symbol Analog Processing-altium-import:3_1uF
- removed C29, C30, C33: (no value), symbol Analog Processing-altium-import:1_100u
- removed C31, C34, C37, C43, C45, C49, C50, C66: (no value), symbol Analog Processing-altium-import:3_10u
- removed C32, C35, C36, C44, C48, C51, C64: (no value), symbol Analog Processing-altium-import:1_0.1u
- removed C38: (no value), symbol Analog Processing-altium-import:3_100u
- removed C39: (no value), symbol Analog Processing-altium-import:0_10n
- removed C40, C41: (no value), symbol Analog Processing-altium-import:0_22pF
- removed C42, C55: (no value), symbol Analog Processing-altium-import:0_10nF
- removed C52, C54: (no value), symbol Analog Processing-altium-import:0_0.1u
- removed C56, C57: (no value), symbol Analog Processing-altium-import:0_1uF
- removed C58: (no value), symbol Analog Processing-altium-import:1_2.2u
- removed C77, C78: (no value), symbol Analog Processing-altium-import:2_0.1u
- removed CN2: (no value), symbol Analog Processing-altium-import:3_5566-02A-210(-TA)
- removed CN3: (no value), symbol Analog Processing-altium-import:0_Z-230010816209
- removed D1: (no value), symbol Analog Processing-altium-import:2_DSS24
- removed F1: (no value), symbol Analog Processing-altium-import:0_BSMD1812-200-30V
- removed LED1, LED2, LED3, LED4, LED5, LED6: (no value), symbol Analog Processing-altium-import:1_19-217/R6C-AL1M2VY/3T
- removed P1: (no value), symbol Analog Processing-altium-import:0_20P-2.54_JTAG
- removed Q1, Q3, Q4, Q5: (no value), symbol Analog Processing-altium-import:0_TIP41A
- removed R1, R2, R34, R35, R50, R51, R66, R67: (no value), symbol Analog Processing-altium-import:0_5.1k
- removed R10, R11, R28, R29, R45, R46, R61, R62: (no value), symbol Analog Processing-altium-import:0_470
- removed R12, R13, R9: (no value), symbol Analog Processing-altium-import:2_33
- removed R14, R22, R39, R55: (no value), symbol Analog Processing-altium-import:2_1M
- removed R15, R24, R41, R57: (no value), symbol Analog Processing-altium-import:1_6.8k
- removed R16, R23, R40, R56: (no value), symbol Analog Processing-altium-import:1_TBD(LOAD)
- removed R17, R21, R38, R54: (no value), symbol Analog Processing-altium-import:0_2k
- removed R18, R19, R36, R44, R52: (no value), symbol Analog Processing-altium-import:3_1M
- removed R20, R33, R37, R53: (no value), symbol Analog Processing-altium-import:1_1m
- removed R25, R42, R58, R6: (no value), symbol Analog Processing-altium-import:0_6.8k
- removed R26, R27, R31, R60, R64, R65, R72, R73, R74, R75, R76, R77, R78, R79, R80, R81: (no value), symbol Analog Processing-altium-import:0_150k
- removed R3: (no value), symbol Analog Processing-altium-import:0_490K
- removed R30, R47, R5, R63: (no value), symbol Analog Processing-altium-import:1_200
- removed R32: (no value), symbol Analog Processing-altium-import:3_120R
- removed R4, R7: (no value), symbol Analog Processing-altium-import:0_33Ω
- removed R43: (no value), symbol Analog Processing-altium-import:0_120R
- removed R48, R59: (no value), symbol Analog Processing-altium-import:1_10k
- removed R49, R8: (no value), symbol Analog Processing-altium-import:1_4.7k
- removed R68, R69, R70, R71: (no value), symbol Analog Processing-altium-import:1_2ohm 5W
- removed R82, R83, R84, R85: (no value), symbol Analog Processing-altium-import:1_1.5k
- removed RN1, RN2, RN3, RN4, RN5: (no value), symbol Analog Processing-altium-import:3_33
- removed SW1: (no value), symbol Analog Processing-altium-import:0_ADCRST
- removed SW2: (no value), symbol Analog Processing-altium-import:0_MCURST
- removed TPI1, TPI2, TPI3, TPI4, TPV1, TPV2, TPV3, TPV4: (no value), symbol Analog Processing-altium-import:1_JUMPER2
- removed U1, U2, U3, U4: (no value), symbol Analog Processing-altium-import:0_LM358BAIDR
- removed U10: (no value), symbol Analog Processing-altium-import:0_STM32F407VGT6
- removed U11: (no value), symbol Analog Processing-altium-import:0_AMS1117-3.3V
- removed U12: (no value), symbol Analog Processing-altium-import:0_TJA1050T/CM,118
- removed U13: (no value), symbol Analog Processing-altium-import:0_AD7606BSTZ-4
- removed U15: (no value), symbol Analog Processing-altium-import:0_URA2405YMD-10WR3_C969031
- removed U16, U18, U19, U20: (no value), symbol Analog Processing-altium-import:0_OPA452FA/500
- removed U17: (no value), symbol Analog Processing-altium-import:0_URA2424YMD-10WR3
- removed U5, U6, U7, U8: (no value), symbol Analog Processing-altium-import:0_URB2409YMD-10WR3
- removed U9: (no value), symbol Analog Processing-altium-import:2_LM4030AMF-2.5/NOPB
- removed X1: (no value), symbol Analog Processing-altium-import:0_DSUB9
- removed Y1: (no value), symbol Analog Processing-altium-import:3_8.000MHZ
- added C1, C15, C16, C2, C25, C26, C4, C5: (no value), CAPC3216X190N, symbol STM32_Mini_Platform_V001_xx_Draft-altium-import:1_CAP_1206_220UF
- added C10, C11, C13, C14, C18, C19, C28, C30, C37, C38, C61: (no value), LC-0603_C, symbol STM32_Mini_Platform_V001_xx_Draft-altium-import:1_CAP_0603_100NF
- added C12, C22, C3, C31: (no value), C1210, symbol STM32_Mini_Platform_V001_xx_Draft-altium-import:1_CAP_1210_22UF
- added C17, C21, C24, C27, C35, C42, C44, C51, C6, C9: (no value), LC-0603_C, symbol STM32_Mini_Platform_V001_xx_Draft-altium-import:0_CAP_0603_100NF
- added C20, C29, C33, C7: (no value), CAP_J-V_8X10P5_RUB, symbol STM32_Mini_Platform_V001_xx_Draft-altium-import:1_50TZV100M8X10.5
- added C23, C34, C43, C56, C57, C8: (no value), CAPPM7343X310N, symbol STM32_Mini_Platform_V001_xx_Draft-altium-import:1_T491D106K050AT
- added C32, C36: (no value), CAPPM7343X310N, symbol STM32_Mini_Platform_V001_xx_Draft-altium-import:0_T491D106K050AT
- added C39, C40: (no value), LC-0603_C, symbol STM32_Mini_Platform_V001_xx_Draft-altium-import:1_CAP_0603_10NF
- added C41, C54: (no value), LC-0603_C, symbol STM32_Mini_Platform_V001_xx_Draft-altium-import:0_CAP_0603_10NF
- added C45, C46: (no value), LC-0603_C, symbol STM32_Mini_Platform_V001_xx_Draft-altium-import:1_CAP_0603_1UF
- added C47, C49, C50: (no value), LC-0603_C, symbol STM32_Mini_Platform_V001_xx_Draft-altium-import:0_CAP_0603_10UF
- added C48: (no value), LC-0603_C, symbol STM32_Mini_Platform_V001_xx_Draft-altium-import:0_CAP_0603_2.2UF
- added C52, C53: (no value), LC-0603_C, symbol STM32_Mini_Platform_V001_xx_Draft-altium-import:1_CAP_0603_16PF
- added C55: (no value), LC-0603_C, symbol STM32_Mini_Platform_V001_xx_Draft-altium-import:0_CAP_0603_1UF
- added C58, C59: (no value), LC-0603_C, symbol STM32_Mini_Platform_V001_xx_Draft-altium-import:2_CAP_0603_100NF
- added C60: (no value), LC-0603_C, symbol STM32_Mini_Platform_V001_xx_Draft-altium-import:1_CAP_0603_10UF
- added CN1: (no value), IDC-SMD_16P-P2.54_Z-S230321016M2BLT1, symbol STM32_Mini_Platform_V001_xx_Draft-altium-import:3_Z-S230321016M2BLT1
- added CN2: (no value), 39-28-8020, symbol STM32_Mini_Platform_V001_xx_Draft-altium-import:0_mirrored_39-28-8020
- added D1, D2, D3, D4, D5, D6: (no value), LED0603-R-RD, symbol STM32_Mini_Platform_V001_xx_Draft-altium-import:1_19-217/R6C-AL1M2VY{slas…
- added D7: (no value), SOD-123FL_L2.7-W1.8-LS3.8-RD, symbol STM32_Mini_Platform_V001_xx_Draft-altium-import:2_DSS24
- added F1: (no value), F1812, symbol STM32_Mini_Platform_V001_xx_Draft-altium-import:0_BSMD1812-200-30V
- added P1: (no value), CONN-SMD_20P-P2.54_B-3000N20P-0110, symbol STM32_Mini_Platform_V001_xx_Draft-altium-import:3_BH-00019
- added Q1, Q2, Q3, Q4: (no value), TO255P460X1020X2008-3P, symbol STM32_Mini_Platform_V001_xx_Draft-altium-import:0_TIP41C
- added R1, R2, R26, R27, R38, R39, R7, R8: (no value), LC-0603_R, symbol STM32_Mini_Platform_V001_xx_Draft-altium-import:0_RES_0603_5.1K
- added R10, R11, R24, R25, R3, R36, R37, R4: (no value), LC-0603_R, symbol STM32_Mini_Platform_V001_xx_Draft-altium-import:0_RES_0603_470
- added R12, R15, R28, R29, R40, R41, R6, R9: (no value), R1210, symbol STM32_Mini_Platform_V001_xx_Draft-altium-import:1_RES_1210_6.8K
- added R13, R18, R30, R42, R56: (no value), LC-0603_R, symbol STM32_Mini_Platform_V001_xx_Draft-altium-import:1_RES_0603_1M
- added R14, R19, R31, R43: (no value), LC-0603_R, symbol STM32_Mini_Platform_V001_xx_Draft-altium-import:3_RES_0603_1M
- added R16, R23, R35, R47: (no value), MF0W4FF6801A50, symbol STM32_Mini_Platform_V001_xx_Draft-altium-import:1_TBD
- added R17, R20, R32, R44: (no value), LC-0603_R, symbol STM32_Mini_Platform_V001_xx_Draft-altium-import:1_RES_0603_2K
- added R21, R33, R45, R67: (no value), RX27-5, symbol STM32_Mini_Platform_V001_xx_Draft-altium-import:1_RX27-5
- added R22, R34, R46, R5: (no value), R2512, symbol STM32_Mini_Platform_V001_xx_Draft-altium-import:1_RES_2512_200
- added R48, R49, R50, R68: (no value), PA2512FKE7W0R001E, symbol STM32_Mini_Platform_V001_xx_Draft-altium-import:1_RES_2512_0.001
- added R51, R52: (no value), LC-0603_R, symbol STM32_Mini_Platform_V001_xx_Draft-altium-import:0_RES_0603_10K
- added R53: (no value), LC-0603_R, symbol STM32_Mini_Platform_V001_xx_Draft-altium-import:0_RES_0603_120
- added R54: (no value), LC-0603_R, symbol STM32_Mini_Platform_V001_xx_Draft-altium-import:1_RES_0603_120
- added R55: (no value), LC-0603_R, symbol STM32_Mini_Platform_V001_xx_Draft-altium-import:0_RES_0603_487K
- added R57, R58, R60, R61: (no value), LC-0603_R, symbol STM32_Mini_Platform_V001_xx_Draft-altium-import:1_RES_0603_33
- added R59: (no value), LC-0603_R, symbol STM32_Mini_Platform_V001_xx_Draft-altium-import:1_mirrored_RES_0603_33
- added R62, R63, R64, R65, R72: (no value), LC-0603_R, symbol STM32_Mini_Platform_V001_xx_Draft-altium-import:0_RES_0603_0R
- added R66, R69, R70, R71: (no value), LC-0603_R, symbol STM32_Mini_Platform_V001_xx_Draft-altium-import:1_RES_0603_1.5K
- added R73, R74, R75, R76, R77, R78, R79, R80, R81, R82, R83, R84, R85, R86, R87, R88: (no value), LC-0603_R, symbol STM32_Mini_Platform_V001_xx_Draft-altium-import:0_RES_0603_150K
- added R89, R90: (no value), LC-0603_R, symbol STM32_Mini_Platform_V001_xx_Draft-altium-import:1_RES_0603_4.7K
- added RN1, RN2: (no value), RES-ARRAY-SMD_0402-8P-L2.0-W1.0-BL, symbol STM32_Mini_Platform_V001_xx_Draft-altium-import:1_mirrored_YC124-FR-0733RL
- added RN3, RN4, RN5: (no value), RES-ARRAY-SMD_0402-8P-L2.0-W1.0-BL, symbol STM32_Mini_Platform_V001_xx_Draft-altium-import:0_mirrored_YC124-FR-0733RL
- added S1, S2: (no value), KEY-SMD_L6.2-W3.6-LS8.0, symbol STM32_Mini_Platform_V001_xx_Draft-altium-import:0_K2-1107ST-A4DW-06
- added TP1: (no value), PAD-1.2, symbol STM32_Mini_Platform_V001_xx_Draft-altium-import:0_mirrored_TP
- added TP2: (no value), PAD-1.2, symbol STM32_Mini_Platform_V001_xx_Draft-altium-import:2_TP
- added TP3, TP4: (no value), PAD-1.2, symbol STM32_Mini_Platform_V001_xx_Draft-altium-import:1_TP
- added TPV1, TPV2, TPV3, TPV4, TPV5, TPV6, TPV7, TPV8: (no value), HDR-SMD_2P-P2.54-V-M-S4.8, symbol STM32_Mini_Platform_V001_xx_Draft-altium-import:0_X6511WVS-02H-C60D48-R1
- added U1: (no value), SOIC127P600X175-8N, symbol STM32_Mini_Platform_V001_xx_Draft-altium-import:0_TJA1050T_CM_118
- added U10, U11, U3, U4: (no value), LM2904BQDRQ1, symbol STM32_Mini_Platform_V001_xx_Draft-altium-import:0_LM2904BQDRQ1
- added U12: (no value), QFP50P1600X1600X160-100N, symbol STM32_Mini_Platform_V001_xx_Draft-altium-import:0_STM32F407VGT6
- added U13, U14, U15, U16: (no value), KTW7, symbol STM32_Mini_Platform_V001_xx_Draft-altium-import:0_OPA452FA/500
- added U17: (no value), SOT95P280X145-5N, symbol STM32_Mini_Platform_V001_xx_Draft-altium-import:0_mirrored_LM4030AMF-2.5_NOPB
- added U18: (no value), SOT-223_L6.5-W3.5-P2.30-LS7.0-BR, symbol STM32_Mini_Platform_V001_xx_Draft-altium-import:0_AMS1117-3.3V
- added U19: (no value), URAXXXXYMD-10WR3, symbol STM32_Mini_Platform_V001_xx_Draft-altium-import:2_URA2405YMD-10WR3
- added U2: (no value), QFP50P1200X1200X160-64N, symbol STM32_Mini_Platform_V001_xx_Draft-altium-import:0_AD7606BSTZ-4
- added U20, U21, U22, U23: (no value), HEATSINK-TH_L23.5-W16.0-P18.0_XSD2156-06, symbol STM32_Mini_Platform_V001_xx_Draft-altium-import:1_23.5X16X25
- added U5, U6, U7, U8: (no value), URBXXXXYMD-10WR3, symbol STM32_Mini_Platform_V001_xx_Draft-altium-import:0_URB2409YMD-10WR3
- added U9: (no value), URAXXXXYMD-10WR3, symbol STM32_Mini_Platform_V001_xx_Draft-altium-import:2_URA2424YMD-10WR3
- added X1: (no value), DSUB-TH_DMR-9S, symbol STM32_Mini_Platform_V001_xx_Draft-altium-import:3_mirrored_D-DMR009PF-D002
- added Y1: (no value), ABLS-12.000MHZ-B2, symbol STM32_Mini_Platform_V001_xx_Draft-altium-import:1_ABLS-8.000MHZ-K4T
Connections:
- net +24V: now also C20.1 (+), C29.1 (+), C33.1 (+), C7.1 (+), D7.1 (C), U19.2 (VIN), U5.2 (VIN), U6.2 (VIN), U7.2 (VIN), U8.2 (VIN), U9.2 (VIN)
- net +3V3: now also C49.1, C54.2, C55.2, P1.1, U12.100 (VDD_6), U12.11 (VDD_1), U12.19 (VDD_2), U12.22 (VDDA), U12.28 (VDD_3), U12.50 (VDD_4), U12.75 (VDD_5), U18.2 (VOUT), U18.4 (VOUT), U2.23 (VDRIVE)
- net +5V: now also C41.2, C42.1, C50.1, C51.1, C56.2, C58.1, C61.1, R55.1, U1.3 (VCC), U18.3 (VIN), U19.3 (+VOUT), U2.1 (AVCC), U2.37 (AVCC), U2.38 (AVCC), U2.48 (AVCC)
- net +9V_1: now also C43.2, C44.2, R66.1, R67.2, U5.3 (_VOUT)
- net +9V_2: now also C34.2, C35.2, R21.2, R70.1, U7.3 (_VOUT)
- net +9V_3: now also C23.2, C24.2, R45.2, R71.1, U8.3 (_VOUT)
- net +9V_4: now also C8.2, C9.2, R33.2, R69.1, U6.3 (_VOUT)
- net -24V: now also C20.2 (-), C29.2 (-), C33.2 (-), C7.2 (-), CN2.1, U19.1 (GND), U5.1 (GND), U6.1 (GND), U7.1 (GND), U8.1 (GND), U9.1 (GND)
- net AD1RST: now also R51.1, U2.11 (RESET)
- net BUSY: now also RN4.5, U2.14 (BUSY)
- net C1A: now also C2.2, R11.2, R74.1
- net C1D: now also R10.1, U12.63 (PC6)
- net C1I: now also R1.1, R76.2, U13.6 (VO)
- net C2A: now also C5.2, R4.2, R78.1
- net C2D: now also R3.1, U12.64 (PC7)
- net C2I: now also R7.1, R80.2, U14.6 (VO)
- net C3A: now also C26.2, R37.2, R82.1
- net C3D: now also R36.1, U12.65 (PC8)
- net C3I: now also R38.1, R84.2, U15.6 (VO)
- net C4: now also C22.2, CN1.1, CN1.2, Q3.3 (E), R34.2, R35.2, TPV6.1, U2.59 (V4)
- net C4A: now also C16.2, R25.2, R86.1
- net C4D: now also R24.1, U12.66 (PC9)
- net C4I: now also R26.1, R88.2, U16.6 (VO)
- net CAN1_RX: now also R54.2, U1.1 (TXD), U12.70 (PA11)
- net CAN1_TX: now also R54.1, U1.4 (RXD), U12.71 (PA12)
- net CONVSTART: now also R57.1, R61.2, U2.10 (CONVST_B), U2.9 (CONVST_A)
- net D0: now also RN3.8, U2.16 (DB0)
- net D1: now also RN3.7, U2.17 (DB1)
- net D10: now also RN1.6, U2.28 (DB10)
- net D11: now also RN1.5, U2.29 (DB11)
- net D12: now also RN2.8, U2.30 (DB12)
- net D13: now also RN2.7, U2.31 (DB13)
- net D14: now also RN2.6, U2.32 (DB14/HBEN)
- net D15: now also RN2.5, U2.33 (DB15/BYTE_SEL)
- net D2: now also RN3.6, U2.18 (DB2)
- net D3: now also RN3.5, U2.19 (DB3)
- net D4: now also RN5.8, U2.20 (DB4)
- net D5: now also RN5.7, U2.21 (DB5)
- net D6: now also RN5.6, U2.22 (DB6)
- net D7: now also RN5.5, U2.24 (DB7/DOUTA)
- net D8: now also RN1.8, U2.25 (DB8/DOUTB)
- net D9: now also RN1.7, U2.27 (DB9)
- net FIRSTDATA: now also R60.2, U2.15 (FRSTDATA)
- net GND: now also C39.2, C40.2, C41.1, C42.2, C46.2, C47.1, C48.2, C49.2, C50.2, C51.2, C52.1, C53.1, C54.1, C55.1, C56.1, C57.2, C58.2, C59.1, C60.2, C61.2, P1.10, P1.12, P1.14, P1.16, P1.18, P1.2, P1.20, P1.4, P1.6, P1.8, R59.2, S1.2, S2.2, U1.2 (GND), U1.8 (S), U12.10 (VSS_1), U12.20 (VSSA), U12.27 (VSS_2), U12.74 (VSS_3), U12.99 (VSS_4), U17.5 (GND), U18.1 (GND), U19.4 (0V), U2.2 (AGND), U2.26 (AGND), U2.3 (OS_0), U2.34 (REF_SELECT), U2.35 (AGND), U2.4 (OS_1), U2.41 (AGND), U2.43 (REFGND), U2.46 (REFGND), U2.47 (AGND), U2.5 (OS_2), U2.53 (AGND), U2.54 (AGND), U2.55 (AGND), U2.56 (AGND), U2.6 (\PA~{R}/SER/BYTE_SEL), U2.61 (AGND), U2.62 (AGND), U2.63 (AGND), U2.64 (AGND), U2.7 (\STBY), U2.8 (RANGE)
- net GND1: now also C13.2, C14.2, C21.2, C43.1, C44.1, CN1.15, CN1.16, D1.2 (C), R15.1, R18.1, R2.1, R48.1, R65.1, R73.1, TPV5.1, U2.50 (V1GND), U3.4 (V-), U5.5 (0V)
- net GND2: now also C10.2, C11.2, C34.1, C35.1, C6.2, CN1.11, CN1.12, D2.2 (C), R13.1, R49.1, R64.1, R77.1, R8.1, R9.1, TPV2.1, U2.52 (V2GND), U4.4 (V-), U7.5 (0V)
- net GND3: now also C23.1, C24.1, C27.2, C28.2, C30.2, CN1.7, CN1.8, D4.2 (C), R39.1, R40.1, R42.1, R63.1, R68.1, R81.1, TPV7.1, U11.4 (V-), U2.58 (V3GND), U8.5 (0V)
- net GND4: now also C17.2, C18.2, C19.2, C8.1, C9.1, CN1.3, CN1.4, D3.2 (C), R27.1, R28.1, R30.1, R50.1, R62.1, R85.1, TPV4.1, U10.4 (V-), U2.60 (V4GND), U6.5 (0V)
- net ISO24V+: now also C32.2, C37.1, R89.2, U13.5 (V+), U14.5 (V+), U15.5 (V+), U16.5 (V+), U9.3 (+VOUT)
- net ISO24V-: now also C36.1, C38.2, D6.2 (C), U13.4 (V-), U14.4 (V-), U15.4 (V-), U16.4 (V-), U9.5 (-VOUT)
- net MCURST: now also R52.1, U12.14 (NRST)
- net PA13: now also P1.7, U12.72 (PA13)
- net PA14: now also P1.9, U12.76 (PA14)
- net PB3: now also P1.13, RN4.8
- net SGND: now also C1.1, C15.1, C16.1, C2.1, C25.1, C26.1, C4.1, C5.1, R72.2
- new net: C22.1, R32.1, R34.1, R35.1, R50.2, TPV6.2
- new net: C53.2, R56.1, U12.13 (PH1), Y1.1 (OSC1)
- new net: C52.2, R56.2, U12.12 (PH0), Y1.2 (OSC2)
- new net: C39.1, R51.2, S1.1
- new net: C28.1, C30.1, Q4.2 (C), R45.1, U11.8 (V+), U22.1, U22.2
- new net: Q2.1 (B), R12.2, U4.1 (OUT1)
- new net: R12.1, R7.2, U4.2 (IN1-)
- new net: C6.1, R8.2, R9.2, U4.3 (IN1+)
- new net: R13.2, U4.5 (IN2+)
- new net: R19.2, R20.2, U4.6 (IN2-)
- new net: R19.1, TPV2.2, U4.7 (OUT2)
- new net: C10.1, C11.1, Q2.2 (C), R21.1, U21.1, U21.2, U4.8 (V+)
- new net: D6.1 (A), R90.1
- new net: C3.1, R16.1, R17.1, R48.2, R5.1, TPV1.2
- new net: C1.2, R10.2, R11.1
- new net: C15.2, R24.2, R25.1
- new net: R1.2, R6.1, U3.2 (IN1-)
- new net: Q1.1 (B), R6.2, U3.1 (OUT1)
- new net: P1.5, TP2.1
- new net: RN2.1, U12.59 (PD12)
- new net: RN2.2, U12.60 (PD13)
- new net: RN2.3, U12.61 (PD14)
- new net: RN2.4, U12.62 (PD15)
- new net: R75.2, R76.1, U13.2 (VIN-)
- new net: R53.1, U1.6 (CANL), X1.2
- new net: R53.2, U1.7 (CANH), X1.7
- new net: C25.2, R36.2, R37.1
- new net: C31.1, R44.1, R46.1, R47.1, R68.2, TPV8.2
- new net: C4.2, R3.2, R4.1
- new net: C12.1, R20.1, R22.1, R23.1, R49.2, TPV3.2
- new net: C17.1, R27.2, R28.2, U10.3 (IN1+)
- new net: Q4.1 (B), R41.2, U11.1 (OUT1)
- new net: R38.2, R41.1, U11.2 (IN1-)
- new net: C27.1, R39.2, R40.2, U11.3 (IN1+)
- new net: R42.2, U11.5 (IN2+)
- new net: R43.2, R44.2, U11.6 (IN2-)
- new net: R43.1, TPV7.2, U11.7 (OUT2)
- new net: R77.2, R78.2, U14.1 (VIN+)
- new net: C57.1, C59.2, U19.5 (-VOUT)
- new net: D2.1 (A), R70.2
- new net: C46.1, U2.36 (REGCAP)
- new net: R79.2, R80.1, U14.2 (VIN-)
- new net: R14.1, TPV5.2, U3.7 (OUT2)
- new net: R14.2, R17.2, U3.6 (IN2-)
- new net: P1.3, TP1.1
- new net: R85.2, R86.2, U16.1 (VIN+)
- new net: R87.2, R88.1, U16.2 (VIN-)
- new net: D3.1 (A), R69.2
- new net: C21.1, R15.2, R2.2, U3.3 (IN1+)
- new net: TP3.1, U12.77 (PA15)
- new net: C40.1, R52.2, S2.1
- new net: R57.2, U12.47 (PB10)
- new net: RN1.1, U12.55 (PD8)
- new net: RN1.2, U12.56 (PD9)
- new net: RN1.3, U12.57 (PD10)
- new net: RN1.4, U12.58 (PD11)
- new net: C13.1, C14.1, Q1.2 (C), R67.1, U20.1, U20.2, U3.8 (V+)
- new net: R73.2, R74.2, U13.1 (VIN+)
- new net: Q3.1 (B), R29.2, U10.1 (OUT1)
- new net: R26.2, R29.1, U10.2 (IN1-)
- new net: R30.2, U10.5 (IN2+)
- new net: R31.2, R32.2, U10.6 (IN2-)
- new net: R31.1, TPV4.2, U10.7 (OUT2)
- new net: C18.1, C19.1, Q3.2 (C), R33.1, U10.8 (V+), U23.1, U23.2
- new net: D1.1 (A), R66.2
- new net: R81.2, R82.2, U15.1 (VIN+)
- new net: R83.2, R84.1, U15.2 (VIN-)
- new net: R18.2, U3.5 (IN2+)
- new net: RN3.1, U12.81 (PD0)
- new net: RN3.2, U12.82 (PD1)
- new net: RN3.3, U12.83 (PD2)
- new net: RN3.4, U12.84 (PD3)
- new net: R60.1, U12.93 (PB7)
- new net: D5.1 (A), R89.1
- new net: CN2.2, F1.1
- new net: R58.2, U12.48 (PB11)
- new net: D7.2 (A), F1.2
- new net: C60.1, U2.44 (REFCAPA), U2.45 (REFCAPB)
- new net: D4.1 (A), R71.2
- new net: RN4.1, U12.89 (PB3)
- new net: RN4.2, U12.90 (PB4)
- new net: RN4.3, U12.91 (PB5)
- new net: RN4.4, U12.92 (PB6)
- new net: RN4.7, TP4.1
- new net: RN5.1, U12.85 (PD4)
- new net: RN5.2, U12.86 (PD5)
- new net: RN5.3, U12.87 (PD6)
- new net: RN5.4, U12.88 (PD7)
- new net: C45.1, U2.40 (AGND)
- new net: C45.2, U2.39 (REGCAP)
- new net: R59.1, U12.96 (PB9)
- new net: R61.1, U12.95 (PB8)
- new net 2V5REF: C47.2, C48.1, R55.2, U17.4 (+VREF), U2.42 (REFIN/REFOUT)
- new net C1: C3.2, CN1.13, CN1.14, Q1.3 (E), R16.2, R5.2, R64.2, TPV1.1, U2.49 (V1)
- new net C2: C12.2, CN1.10, CN1.9, Q2.3 (E), R22.2, R23.2, R63.2, TPV3.1, U2.51 (V2)
- new net C3: C31.2, CN1.5, CN1.6, Q4.3 (E), R46.2, R47.2, R62.2, TPV8.1, U2.57 (V3)
- new net CHIPSELECT#: RN4.6, U2.13 (\CS)
- new net EPAD: U13.8 (EPAD), U14.8 (EPAD), U15.8 (EPAD), U16.8 (EPAD)
- new net ISOGND: C32.1, C36.2, C37.2, C38.1, D5.2 (C), R65.2, R72.1, R75.1, R79.1, R83.1, R87.1, R90.2, U9.4 (0V)
- new net READDATA#: R58.1, U2.12 (\R~{D}/SCLK)
- no-connect marks 1 -> 0
Other:
- note removed: "24V Isolation"
- note removed: "2V5 Reference Voltage With Calibration"
- note removed: "3V3 VOLTAGE"
- note removed: "5V Power Supply"
- note removed: "MCU"
- note removed: "PGND TO SGND"
- note removed: "Signals I/O"
- note removed: "VOLTAGE OUTPUT"
- title: (none) -> AL_CSA_Platform

Commit message: Refactoring and CAN Fix:   * refactoring overlapped net lebels around MCU and ADC   * remove MCU-side 120ohm resister on CAN Tranceiver   * fix: swap CAN RX/TX   * fix: PA11/12 <----> PB5/6
Parts:
- removed R54: (no value), LC-0603_R, symbol STM32_Mini_Platform_V001_xx_Draft-altium-import:1_RES_0603_120
- C1, C15, C16, C2, C25, C26, C4, C5: value (none) -> CAP_1206_220UF
- C10, C11, C13, C14, C17, C18, C19, C21, C24, C27, C28, C30, C35, C37, C38, C42, C44, C51, C58, C59, C6, C61, C9: value (none) -> CAP_0603_100NF
- C12, C22, C3, C31: value (none) -> CAP_1210_22UF
- C20, C29, C33, C7: value (none) -> 50TZV100M8X10.5
- C23, C32, C34, C36, C43, C56, C57, C8: value (none) -> T491D106K050AT
- C39, C40, C41, C54: value (none) -> CAP_0603_10NF
- C45, C46, C55: value (none) -> CAP_0603_1UF
- C47, C49, C50, C60: value (none) -> CAP_0603_10UF
- C48: value (none) -> CAP_0603_2.2UF
- C52, C53: value (none) -> CAP_0603_16PF
- CN1: value (none) -> Z-S230321016M2BLT1
- CN2: value (none) -> 39-28-8020
- D1, D2, D3, D4, D5, D6: value (none) -> 19-217/R6C-AL1M2VY/3T
- D7: value (none) -> DSS24
- F1: value (none) -> BSMD1812-200-30V
- P1: value (none) -> BH-00019
- Q1, Q2, Q3, Q4: value (none) -> TIP41C
- R1, R2, R26, R27, R38, R39, R7, R8: value (none) -> RES_0603_5.1K
- R10, R11, R24, R25, R3, R36, R37, R4: value (none) -> RES_0603_470
- R12, R15, R28, R29, R40, R41, R6, R9: value (none) -> RES_1210_6.8K
- R13, R14, R18, R19, R30, R31, R42, R43, R56: value (none) -> RES_0603_1M
- R16, R23, R35, R47: value (none) -> TBD
- R17, R20, R32, R44: value (none) -> RES_0603_2K
- R21, R33, R45, R67: value (none) -> RX27-5
- R22, R34, R46, R5: value (none) -> RES_2512_200
- R48, R49, R50, R68: value (none) -> RES_2512_0.001
- R51, R52: value (none) -> RES_0603_10K
- R53: value (none) -> RES_0603_120
- R55: value (none) -> RES_0603_487K
- R57, R58, R59, R60, R61: value (none) -> RES_0603_33
- R62, R63, R64, R65, R72: value (none) -> RES_0603_0R
- R66, R69, R70, R71: value (none) -> RES_0603_1.5K
- R73, R74, R75, R76, R77, R78, R79, R80, R81, R82, R83, R84, R85, R86, R87, R88: value (none) -> RES_0603_150K
- R89, R90: value (none) -> RES_0603_4.7K
- RN1, RN2, RN3, RN4, RN5: value (none) -> YC124-FR-0733RL
- S1, S2: value (none) -> K2-1107ST-A4DW-06
- TP1, TP2, TP3, TP4: value (none) -> TP
- TPV1, TPV2, TPV3, TPV4, TPV5, TPV6, TPV7, TPV8: value (none) -> X6511WVS-02H-C60D48-R1
- U1: value (none) -> TJA1050T_CM_118
- U10, U11, U3, U4: value (none) -> LM2904BQDRQ1
- U12: value (none) -> STM32F407VGT6
- U13, U14, U15, U16: value (none) -> OPA452FA/500
- U17: value (none) -> LM4030AMF-2.5_NOPB
- U18: value (none) -> AMS1117-3.3V
- U19: value (none) -> URA2405YMD-10WR3
- U2: value (none) -> AD7606BSTZ-4
- U20, U21, U22, U23: value (none) -> 23.5X16X25
- U5, U6, U7, U8: value (none) -> URB2409YMD-10WR3
- U9: value (none) -> URA2424YMD-10WR3
- X1: value (none) -> D-DMR009PF-D002
- Y1: value (none) -> ABLS-8.000MHZ-K4T
Connections:
- net BUSY: now also U12.71 (PA12); no longer RN4.5
- net CAN1_RX: now also RN4.6, U1.4 (RXD); no longer U1.1 (TXD), U12.70 (PA11)
- net CAN1_TX: now also RN4.5, U1.1 (TXD); no longer U1.4 (RXD), U12.71 (PA12)
- net CHIPSELECT#: now also U12.70 (PA11); no longer RN4.6
- net GND: no longer R59.2, U2.7 (\STBY)
- new net STANDBY#: R59.2, U2.7 (\STBY)
Other:
- moved on the sheet: C46, R62, R63, R64, R65, RN3, RN4, RN5, TP4

Commit message: update OP amp circuit, update PCB.
Parts:
- removed R1, R26, R38, R7: RES_0603_5.1K, LC-0603_R, symbol STM32_Mini_Platform_V001_xx_Draft-altium-import:0_RES_0603_5.1K
- removed R15, R28, R40, R9: RES_1210_6.8K, R1210, symbol STM32_Mini_Platform_V001_xx_Draft-altium-import:1_RES_1210_6.8K
- R12, R29, R6: ALTIUM_VALUE 6.8k -> 10k
- R2, R27, R8: ALTIUM_VALUE 5.1K -> 10K
- U10, U11, U3, U4: value LM2904BQDRQ1 -> (none)
Connections:
- net C1: now also R6.2
- net C1I: now also R2.1
- net C2: now also R12.2
- net C2I: now also R8.1
- net C3: now also R41.2
- net C3I: now also R39.1
- net C4: now also R29.2
- net C4I: now also R27.1
- net GND1: no longer R2.1
- net GND2: no longer R8.1
- net GND3: no longer R39.1
- net GND4: no longer R27.1
- net at Q2.1 (B), U4.1 (OUT1): no longer R12.2
- net at Q1.1 (B), U3.1 (OUT1): no longer R6.2
- net at Q4.1 (B), U11.1 (OUT1): no longer R41.2
- net at Q3.1 (B), U10.1 (OUT1): no longer R29.2

Commit message: add FIU relay schematics.
Parts:
- added D11: (no value), symbol SS34:SS34
- added D12, D13, D21, D22, D23, D31, D32, D33, D41, D42, D43: SS34, DIOM7959X265N, symbol SS34:SS34
- added Q11: (no value), symbol Transistor_FET:AO3400A
- added Q12, Q13, Q21, Q22, Q23, Q31, Q32, Q33, Q41, Q42, Q43: AO3400A, Package_TO_SOT_SMD:SOT-23, symbol Transistor_FET:AO3400A
- added RL11: (no value), symbol V23105A5001A201:V23105A5001A201
- added RL12, RL13, RL21, RL22, RL23, RL31, RL32, RL33, RL41, RL42, RL43: V23105A5001A201, RELAY8-398X799_451, symbol V23105A5001A201:V23105A5001A201
- U10, U11, U3, U4: value (none) -> OPA2202
Connections:
- net +5V: now also D11.C, D12.C, D13.C, D21.C, D22.C, D23.C, D31.C, D32.C, D33.C, D41.C, D42.C, D43.C, RL11.A1, RL12.A1, RL13.A1, RL21.A1, RL22.A1, RL23.A1, RL31.A1, RL32.A1, RL33.A1, RL41.A1, RL42.A1, RL43.A1
- net C1: now also RL11.14, RL12.11
- net C2: now also RL21.14, RL22.11
- net C3: now also RL31.14, RL32.11
- net C4: now also RL41.14, RL42.11
- net GND: now also Q11.2 (S), Q12.2 (S), Q13.2 (S), Q21.2 (S), Q22.2 (S), Q23.2 (S), Q31.2 (S), Q32.2 (S), Q33.2 (S), Q41.2 (S), Q42.2 (S), Q43.2 (S)
- net GND1: now also RL11.24, RL13.11
- net GND2: now also RL21.24, RL23.11
- net GND3: now also RL31.24, RL33.11
- net GND4: now also RL41.24, RL43.11
- net C4_FIU_OC: now reaches U12.30 (PA5)
- net C4_FIU_OC: now also Q41.1 (G)
- net C4_FIU_SC1: now reaches U12.31 (PA6)
- net C4_FIU_SC1: now also Q42.1 (G)
- net C4_FIU_SC2: now reaches U12.32 (PA7)
- net C4_FIU_SC2: now also Q43.1 (G)
- net C1_FIU_OC: now reaches U12.38 (PE7)
- net C1_FIU_OC: now also Q11.1 (G)
- net C1_FIU_SC1: now reaches U12.39 (PE8)
- net C1_FIU_SC1: now also Q12.1 (G)
- net C1_FIU_SC2: now reaches U12.40 (PE9)
- net C1_FIU_SC2: now also Q13.1 (G)
- net C2_FIU_OC: now reaches U12.41 (PE10)
- net C2_FIU_OC: now also Q21.1 (G)
- net C2_FIU_SC1: now reaches U12.42 (PE11)
- net C2_FIU_SC1: now also Q22.1 (G)
- net C2_FIU_SC2: now reaches U12.43 (PE12)
- net C2_FIU_SC2: now also Q23.1 (G)
- net C3_FIU_OC: now reaches U12.44 (PE13)
- net C3_FIU_OC: now also Q31.1 (G)
- net C3_FIU_SC1: now reaches U12.45 (PE14)
- net C3_FIU_SC1: now also Q32.1 (G)
- net C3_FIU_SC2: now reaches U12.46 (PE15)
- net C3_FIU_SC2: now also Q33.1 (G)
- new net: D22.A, Q22.3 (D), RL22.A2
- new net: D12.A, Q12.3 (D), RL12.A2
- new net: RL11.11, RL12.14, RL13.12
- new net: RL11.21, RL12.12, RL13.14
- new net: D13.A, Q13.3 (D), RL13.A2
- new net: RL31.21, RL32.12, RL33.14
- new net: RL31.11, RL32.14, RL33.12
- new net: D32.A, Q32.3 (D), RL32.A2
- new net: D31.A, Q31.3 (D), RL31.A2
- new net: D33.A, Q33.3 (D), RL33.A2
- new net: D11.A, Q11.3 (D), RL11.A2
- new net: D41.A, Q41.3 (D), RL41.A2
- new net: D42.A, Q42.3 (D), RL42.A2
- new net: RL41.21, RL42.12, RL43.14
- new net: RL41.11, RL42.14, RL43.12
- new net: D43.A, Q43.3 (D), RL43.A2
- new net: D21.A, Q21.3 (D), RL21.A2
- new net: RL21.11, RL22.14, RL23.12
- new net: RL21.21, RL22.12, RL23.14
- new net: D23.A, Q23.3 (D), RL23.A2
Other:
- moved on the sheet: CN1, R57, R58, R62, R63, R64, R65

Commit message: update PCB.
Parts:
- added R_VL1: RES_2512_200, R2512, symbol STM32_Mini_Platform_V001_xx_Draft-altium-import:1_RES_2512_200
Connections:
- net C1_FIU_OC: now also U12.3 (PE4); no longer U12.38 (PE7)
- net C1_FIU_SC1: now also U12.4 (PE5); no longer U12.39 (PE8)
- net C1_FIU_SC2: now also U12.5 (PE6); no longer U12.40 (PE9)
- net C2_FIU_OC: now also U12.38 (PE7); no longer U12.41 (PE10)
- net C2_FIU_SC1: now also U12.39 (PE8); no longer U12.42 (PE11)
- net C2_FIU_SC2: now also U12.40 (PE9); no longer U12.43 (PE12)
- net C3_FIU_OC: now also U12.41 (PE10); no longer U12.44 (PE13)
- net C3_FIU_SC1: now also U12.42 (PE11); no longer U12.45 (PE14)
- net C3_FIU_SC2: now also U12.43 (PE12); no longer U12.46 (PE15)
- net C4_FIU_OC: now also U12.44 (PE13); no longer U12.30 (PA5)
- net C4_FIU_SC1: now also U12.45 (PE14); no longer U12.31 (PA6)
- net C4_FIU_SC2: now also U12.46 (PE15); no longer U12.32 (PA7)
- net GND: now also R_VL1.1
- net Q22C: now reaches D22.A, Q22.3 (D), RL22.A2
- net at C57.1, C59.2, U19.5 (-VOUT): now also R_VL1.2
- net Q12C: now reaches D12.A, Q12.3 (D), RL12.A2
- net C1_: now reaches RL11.11, RL12.14, RL13.12
- net GND1_: now reaches RL11.21, RL12.12, RL13.14
- net Q13C: now reaches D13.A, Q13.3 (D), RL13.A2
- net GND3_: now reaches RL31.21, RL32.12, RL33.14
- net C3_: now reaches RL31.11, RL32.14, RL33.12
- net Q32C: now reaches D32.A, Q32.3 (D), RL32.A2
- net Q31C: now reaches D31.A, Q31.3 (D), RL31.A2
- net Q33C: now reaches D33.A, Q33.3 (D), RL33.A2
- net Q11C: now reaches D11.A, Q11.3 (D), RL11.A2
- net Q41C: now reaches D41.A, Q41.3 (D), RL41.A2
- net Q42C: now reaches D42.A, Q42.3 (D), RL42.A2
- net GND4_: now reaches RL41.21, RL42.12, RL43.14
- net C4_: now reaches RL41.11, RL42.14, RL43.12
- net Q43C: now reaches D43.A, Q43.3 (D), RL43.A2
- net Q21C: now reaches D21.A, Q21.3 (D), RL21.A2
- net C2_: now reaches RL21.11, RL22.14, RL23.12
- net GND2_: now reaches RL21.21, RL22.12, RL23.14
- net Q23C: now reaches D23.A, Q23.3 (D), RL23.A2
Other:
- moved on the sheet: CN1, R62, R63, R64, R65
