File: hardware/cell-simulator.kicad_sch (KiCad schematic)
At the start: 238 parts, among them CN1 Z-S230321016M2BLT1, CN2 39-28-8020, P1 BH-00019, Q1 TIP41C, Q12 AO3400A, Q13 AO3400A, Q2 TIP41C, Q21 AO3400A, Q22 AO3400A, Q23 AO3400A, Q3 TIP41C, Q31 AO3400A, Q32 AO3400A, Q33 AO3400A, Q4 TIP41C, Q41 AO3400A, Q42 AO3400A, Q43 AO3400A, U1 TJA1050T_CM_118, U10 OPA2202, U11 OPA2202, U12 STM32F407VGT6, U13 OPA452FA/500, U14 OPA452FA/500, U15 OPA452FA/500, U16 OPA452FA/500, U17 LM4030AMF-2.5_NOPB, U18 AMS1117-3.3V, U19 URA2405YMD-10WR3, U2 AD7606BSTZ-4, U20 23.5X16X25, U21 23.5X16X25, U22 23.5X16X25, U23 23.5X16X25, U3 OPA2202, U4 OPA2202, U5 URB2409YMD-10WR3, U6 URB2409YMD-10WR3, U7 URB2409YMD-10WR3, U8 URB2409YMD-10WR3, U9 URA2424YMD-10WR3, X1 D-DMR009PF-D002, Y1 ABLS-8.000MHZ-K4T

Commit message: update Sch and PCB: fix MCURST, remove A1RST, fix ADC inputs, improve mounting holes.
Parts:
- removed C39: CAP_0603_10NF, LC-0603_C, symbol STM32_Mini_Platform_V001_xx_Draft-altium-import:1_CAP_0603_10NF
- removed R51: RES_0603_10K, LC-0603_R, symbol STM32_Mini_Platform_V001_xx_Draft-altium-import:0_RES_0603_10K
- removed S1: K2-1107ST-A4DW-06, KEY-SMD_L6.2-W3.6-LS8.0, symbol STM32_Mini_Platform_V001_xx_Draft-altium-import:0_K2-1107ST-A4DW-06
- D11: value (none) -> SS34; footprint (none) -> DIOM7959X265N
- Q11: value (none) -> AO3400A; footprint (none) -> Package_TO_SOT_SMD:SOT-23
- RL11: value (none) -> V23105A5001A201; footprint (none) -> RELAY8-398X799_451
Connections:
- net +3V3: now also R52.2
- net GND: no longer P1.2
- net MCURST: now also C40.1, S2.1
Other:
- moved on the sheet: R52
